File: ThumbLight.kicad_pcb (KiCad board)
At the start: 2 copper layers, 33 x 49 mm, 12 parts, among them J1 USB_A, SW1 RESET, SW2 RESET, SW3 RESET, SW4 RESET, U1 DHT11, U2 UA78M33_TO252, U3 ESP-12E, U4 TTL

Commit message: Silkscreen
Parts:
- SW2: value RESET -> A
- SW3: value RESET -> B
- SW4: value RESET -> MODE
- moved R2 0.88 mm to (95.9, 101.0)
- moved LIN1 0.54 mm to (87.0, 94.0)
- moved SW1 0.40 mm to (86.6, 118.5)
Routing:
- net GND: track 14.0 -> 33.9 mm
- net Net-(U3-Pad2): track 25.4 -> 26.8 mm
- net NEOPIXEL: track 18.2 -> 18.8 mm
Changed lines of the file:
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@@
   )
   (footprint "Resistor_THT:R_Axial_DIN0207_L6.3mm_D2.5mm_P7.62mm_Horizontal" (layer "F.Cu")
-    (at 96.81 101 180)
+    (at 95.930862 101 180)
     (descr "Resistor, Axial_DIN0207 series, Axial, Horizontal, pin pitch=7.62mm, 0.25W = 1/4W, length*diameter=6.3*2.5mm^2, http://cdn-reichelt.de/documents/datenblatt/B400/1_4W%23YAG.pdf")
     (tags "Resistor Axial_DIN0207 series Axial Horizontal pin pitch 7.62mm 0.25W = 1/4W length 6.3mm diameter 2.5mm")
@@
   )
   (footprint "Button_Switch_SMD:SW_Push_1P1T_NO_Vertical_Wuerth_434133025816" (layer "B.Cu")
-    (at 86.47762 118.931768 180)
+    (at 86.576497 118.54799 180)
     (descr "https://katalog.we-online.com/em/datasheet/434133025816.pdf")
     (tags "tactile switch Wurth Wuerth")
@@
     (property "Sheetname" "")
     (attr smd)
-    (fp_text reference "SW2" (at 0.15 2.6 90) (layer "B.SilkS")
-      (effects (font (size 1 1) (thickness 0.15)) (justify mirror))
-    )
-    (fp_text value "RESET" (at 0 -2.55 90) (layer "B.Fab")
+    (fp_text reference "SW2" (at 0.15 2.6 90) (layer "B.SilkS") hide
+      (effects (font (size 1 1) (thickness 0.15)) (justify mirror))
+    )
+    (fp_text value "A" (at 0 -2.55 90) (layer "B.SilkS")
       (effects (font (size 1 1) (thickness 0.15)) (justify mirror))
     )
@@
     (property "Sheetname" "")
     (attr smd)
-    (fp_text reference "SW3" (at 0.15 2.6 90) (layer "B.SilkS")
-      (effects (font (size 1 1) (thickness 0.15)) (justify mirror))
-    )
-    (fp_text value "RESET" (at 0 -2.55 90) (layer "B.Fab")
+    (fp_text reference "SW3" (at 0.15 2.6 90) (layer "B.SilkS") hide
+      (effects (font (size 1 1) (thickness 0.15)) (justify mirror))
+    )
+    (fp_text value "B" (at 0 -2.55 90) (layer "B.SilkS")
       (effects (font (size 1 1) (thickness 0.15)) (justify mirror))
     )
@@
   )
   (footprint "neopixel-strip:neopixel-strip" (layer "B.Cu")
-    (at 87.544466 94.04218 -90)
+    (at 87 94.04218 -90)
     (property "Sheetfile" "ThumbLight.kicad_sch")
     (property "Sheetname" "")
@@
       (effects (font (size 1 1) (thickness 0.15)) (justify mirror))
     )
-    (fp_text value "RESET" (at 0 -2.55 90) (layer "B.Fab")
+    (fp_text value "MODE" (at 0 -2.55 90) (layer "B.Fab")
       (effects (font (size 1 1) (thickness 0.15)) (justify mirror))
     )
@@
     (effects (font (size 1.5 1.5) (thickness 0.3)))
   )
+  (segment (start 84 116.971493) (end 84 113.075) (width 0.6) (layer "B.Cu") (net 1))
+  (segment (start 84 108.925) (end 84 113.075) (width 0.6) (layer "B.Cu") (net 1))
+  (segment (start 84.501497 117.47299) (end 84 116.971493) (width 0.6) (layer "B.Cu") (net 1))
   (segment (start 94.12 82.02) (end 94.12 82.78) (width 0.6) (layer "B.Cu") (net 1))
   (segment (start 94.12 82.78) (end 91.9 85) (width 0.6) (layer "B.Cu") (net 1))
+  (segment (start 84 101.925) (end 84 113.075) (width 0.6) (layer "B.Cu") (net 1))
   (segment (start 96.19 79.95) (end 94.12 82.02) (width 0.6) (layer "B.Cu") (net 1))
-  (segment (start 88.55262 117.856768) (end 84.40262 117.856768) (width 0.6) (layer "B.Cu") (net 1))
+  (segment (start 88.651497 117.47299) (end 84.501497 117.47299) (width 0.6) (layer "B.Cu") (net 1))
   (segment (start 96.19 76.9) (end 96.19 79.95) (width 0.6) (layer "B.Cu") (net 1))
   (segment (start 113 84) (end 112 83) (width 0.6) (layer "F.Cu") (net 2))
@@
   (via (at 86.624255 84) (size 2.5) (drill 0.8) (layers "F.Cu" "B.Cu") (net 2))
   (via (at 113 84) (size 2.5) (drill 0.8) (layers "F.Cu" "B.Cu") (net 2))
-  (segment (start 87 89.941714) (end 87 84.375745) (width 0.6) (layer "B.Cu") (net 2))
-  (segment (start 87.544466 90.48618) (end 87 89.941714) (width 0.6) (layer "B.Cu") (net 2))
+  (segment (start 93.399501 104.500499) (end 93.399501 97.600499) (width 0.6) (layer "B.Cu") (net 2))
+  (segment (start 92.4 105.5) (end 93.399501 104.500499) (width 0.6) (layer "B.Cu") (net 2))
   (segment (start 109 93) (end 110 93) (width 0.6) (layer "B.Cu") (net 2))
   (segment (start 92.4 105.5) (end 94.600499 105.5) (width 0.6) (layer "B.Cu") (net 2))
+  (segment (start 95 97) (end 94 97) (width 0.6) (layer "B.Cu") (net 2))
+  (segment (start 87 90.48618) (end 92.48618 90.48618) (width 0.6) (layer "B.Cu") (net 2))
   (segment (start 94.600499 105.5) (end 96 106.899501) (width 0.6) (layer "B.Cu") (net 2))
   (segment (start 112.025 112.022535) (end 112.317294 112.314829) (width 0.6) (layer "B.Cu") (net 2))
-  (segment (start 92.4 105.5) (end 93 104.9) (width 0.6) (layer "B.Cu") (net 2))
+  (segment (start 93.399501 91.399501) (end 92.48618 90.48618) (width 0.6) (layer "B.Cu") (net 2))
   (segment (start 96 114.100499) (end 94.600499 115.5) (width 0.6) (layer "B.Cu") (net 2))
-  (segment (start 87.544466 90.48618) (end 92.48618 90.48618) (width 0.6) (layer "B.Cu") (net 2))
   (segment (start 112.025 95.025) (end 112.025 112.022535) (width 0.6) (layer "B.Cu") (net 2))
-  (segment (start 93 104.9) (end 93 91) (width 0.6) (layer "B.Cu") (net 2))
-  (segment (start 95 97) (end 93 99) (width 0.6) (layer "B.Cu") (net 2))
+  (segment (start 86 84.624255) (end 86.624255 84) (width 0.6) (layer "B.Cu") (net 2))
   (segment (start 94.99382 90.48618) (end 92.48618 90.48618) (width 0.6) (layer "B.Cu") (net 2))
+  (segment (start 87 90.48618) (end 86 89.48618) (width 0.6) (layer "B.Cu") (net 2))
   (segment (start 98.2 87.28) (end 94.99382 90.48618) (width 0.6) (layer "B.Cu") (net 2))
-  (segment (start 87 84.375745) (end 86.624255 84) (width 0.6) (layer "B.Cu") (net 2))
+  (segment (start 93.399501 97.600499) (end 93.399501 91.399501) (width 0.6) (layer "B.Cu") (net 2))
   (segment (start 112.999999 90.867717) (end 113 84) (width 0.6) (layer "B.Cu") (net 2))
-  (segment (start 92.48618 90.48618) (end 93 91) (width 0.6) (layer "B.Cu") (net 2))
+  (segment (start 86 89.48618) (end 86 84.624255) (width 0.6) (layer "B.Cu") (net 2))
   (segment (start 110.867716 93) (end 112.999999 90.867717) (width 0.6) (layer "B.Cu") (net 2))
   (segment (start 110 93) (end 112.025 95.025) (width 0.6) (layer "B.Cu") (net 2))
   (segment (start 109 93) (end 110.867716 93) (width 0.6) (layer "B.Cu") (net 2))
   (segment (start 94.600499 115.5) (end 92.4 115.5) (width 0.6) (layer "B.Cu") (net 2))
+  (segment (start 94 97) (end 93.399501 97.600499) (width 0.6) (layer "B.Cu") (net 2))
   (segment (start 96 106.899501) (end 96 114.100499) (width 0.6) (layer "B.Cu") (net 2))
-  (segment (start 88.55262 120.006768) (end 91.893232 120.006768) (width 0.6) (layer "B.Cu") (net 3))
-  (segment (start 91.893232 120.006768) (end 92.4 119.5) (width 0.6) (layer "B.Cu") (net 3))
-  (segment (start 84.42762 120.006768) (end 88.55262 120.006768) (width 0.6) (layer "B.Cu") (net 3))
-  (segment (start 96.81 101) (end 96.81 98.19) (width 0.6) (layer "B.Cu") (net 4))
-  (segment (start 97.609999 115.569194) (end 97.609999 101.799999) (width 0.6) (layer "B.Cu") (net 4))
-  (segment (start 96.81 98.19) (end 98 97) (width 0.6) (layer "B.Cu") (net 4))
-  (segment (start 95.679193 117.5) (end 97.609999 115.569194) (width 0.6) (layer "B.Cu") (net 4))
-  (segment (start 97.609999 101.799999) (end 96.81 101) (width 0.6) (layer "B.Cu") (net 4))
+  (segment (start 84.526497 119.62299) (end 88.651497 119.62299) (width 0.6) (layer "B.Cu") (net 3))
+  (segment (start 88.651497 119.62299) (end 92.27701 119.62299) (width 0.6) (layer "B.Cu") (net 3))
+  (segment (start 92.27701 119.62299) (end 92.4 119.5) (width 0.6) (layer "B.Cu") (net 3))
+  (segment (start 95.930862 101) (end 98 101) (width 0.6) (layer "B.Cu") (net 4))
   (segment (start 92.4 117.5) (end 95.679193 117.5) (width 0.6) (layer "B.Cu") (net 4))
+  (segment (start 95.679193 117.5) (end 98 115.179193) (width 0.6) (layer "B.Cu") (net 4))
+  (segment (start 98 115.179193) (end 98 101) (width 0.6) (layer "B.Cu") (net 4))
+  (segment (start 98 101) (end 98 97) (width 0.6) (layer "B.Cu") (net 4))
   (segment (start 86.15 113.05) (end 86.6 113.5) (width 0.6) (layer "B.Cu") (net 5))
   (segment (start 86.6 113.5) (end 92.4 113.5) (width 0.6) (layer "B.Cu") (net 5))
@@
   (segment (start 105.3 113.5) (end 104.3495 112.5495) (width 0.6) (layer "B.Cu") (net 15))
   (segment (start 107.6 113.5) (end 105.3 113.5) (width 0.6) (layer "B.Cu") (net 15))
-  (segment (start 88.620466 94.04218) (end 87.544466 94.04218) (width 0.6) (layer "B.Cu") (net 16))
+  (segment (start 89.8 106.82151) (end 89.8 104.2) (width 0.6) (layer "B.Cu") (net 16))
+  (segment (start 88.620466 94.04218) (end 87 94.04218) (width 0.6) (layer "B.Cu") (net 16))
+  (segment (start 89.8 104.2) (end 91.097494 102.902506) (width 0.6) (layer "B.Cu") (net 16))
+  (segment (start 91.097494 96.519208) (end 88.620466 94.04218) (width 0.6) (layer "B.Cu") (net 16))
   (segment (start 92.4 107.5) (end 90.47849 107.5) (width 0.6) (layer "B.Cu") (net 16))
-  (segment (start 89.8 103.8) (end 91 102.6) (width 0.6) (layer "B.Cu") (net 16))
-  (segment (start 91 96.421714) (end 88.620466 94.04218) (width 0.6) (layer "B.Cu") (net 16))
   (segment (start 90.47849 107.5) (end 89.8 106.82151) (width 0.6) (layer "B.Cu") (net 16))
-  (segment (start 89.8 106.82151) (end 89.8 103.8) (width 0.6) (layer "B.Cu") (net 16))
-  (segment (start 91 102.6) (end 91 96.421714) (width 0.6) (layer "B.Cu") (net 16))
+  (segment (start 91.097494 102.902506) (end 91.097494 96.519208) (width 0.6) (layer "B.Cu") (net 16))
   (segment (start 109.26603 111.5) (end 110.2 110.56603) (width 0.6) (layer "B.Cu") (net 17))
   (segment (start 107.6 111.5) (end 109.26603 111.5) (width 0.6) (layer "B.Cu") (net 17))
