File: ThumbLight.kicad_pcb (KiCad board)
At the start: 2 copper layers, 33 x 53 mm, 12 parts, among them J1 USB_A, SW1 RESET, SW2 A, SW3 B, SW4 MODE, U1 DHT11, U2 UA78M33_TO252, U3 ESP-12E, U4 TTL

Commit message: Update todos
Other:
- board text added: "TODO: - Neopixel needs more space and flat underground - Switches pads need to move to the outside of the switch - Fix DHT11 - Neopixel add header 3 x connector"
- board text removed: "TODO: - Neopixel needs more space and flat underground - Switches pads need to move to the outside of the switch"
Changed lines of the file:
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@@
     (effects (font (size 1.5 1.5) (thickness 0.3)) (justify left))
   )
-  (gr_text "TODO:\n\n- Neopixel needs more space and flat underground\n- Switches pads need to move to the outside of the switch" (at 73 50) (layer "F.Fab")
+  (gr_text "TODO:\n\n- Neopixel needs more space and flat underground\n- Switches pads need to move to the outside of the switch\n- Fix DHT11\n- Neopixel add header 3 x connector \n" (at 73 50) (layer "F.Fab")
     (effects (font (size 1.5 1.5) (thickness 0.3)) (justify left))
   )
